File: clouds_v30.sch (EAGLE design)
At the start: 148 parts, among them IC1 74HC595D, IC10 TL072D, IC2 LM1117-3.3, IC3 MCP6002, IC4 MCP6004, IC5 STM32F405RGT6, IC6 LM4040B10, IC7 LM1117-3.3, IC8 WM8731, IC9 TL072D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

Commit message: moving stuff around, think i should move the i2s interface
Parts:
- renumbered SD to SPI
Changed lines of the file:
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@@
 <part name="ORIG_MAP" library="pinhead" deviceset="PINHD-2X6" device=""/>
 <part name="NEW_MAP" library="pinhead" deviceset="PINHD-1X6" device=""/>
-<part name="SD" library="pinhead" deviceset="PINHD-1X6" device=""/>
+<part name="SPI" library="pinhead" deviceset="PINHD-1X6" device=""/>
 </parts>
 <sheets>
@@
 <instance part="ORIG_MAP" gate="A" x="142.24" y="-25.4"/>
 <instance part="NEW_MAP" gate="A" x="142.24" y="-50.8"/>
-<instance part="SD" gate="A" x="106.68" y="-50.8"/>
+<instance part="SPI" gate="A" x="106.68" y="-50.8"/>
 </instances>
 <busses>
@@
 </segment>
 <segment>
-<pinref part="SD" gate="A" pin="2"/>
+<pinref part="SPI" gate="A" pin="2"/>
 <wire x1="96.52" y1="-45.72" x2="104.14" y2="-45.72" width="0.1524" layer="91"/>
 <label x="88.9" y="-45.72" size="1.778" layer="95"/>
@@
 </segment>
 <segment>
-<pinref part="SD" gate="A" pin="1"/>
+<pinref part="SPI" gate="A" pin="1"/>
 <wire x1="96.52" y1="-43.18" x2="104.14" y2="-43.18" width="0.1524" layer="91"/>
 <label x="88.9" y="-43.18" size="1.778" layer="95"/>
@@
 </segment>
 <segment>
-<pinref part="SD" gate="A" pin="3"/>
+<pinref part="SPI" gate="A" pin="3"/>
 <wire x1="96.52" y1="-48.26" x2="104.14" y2="-48.26" width="0.1524" layer="91"/>
 <label x="88.9" y="-48.26" size="1.778" layer="95"/>
@@
 </segment>
 <segment>
-<pinref part="SD" gate="A" pin="4"/>
+<pinref part="SPI" gate="A" pin="4"/>
 <wire x1="96.52" y1="-50.8" x2="104.14" y2="-50.8" width="0.1524" layer="91"/>
 <label x="88.9" y="-50.8" size="1.778" layer="95"/>
@@
 </segment>
 <segment>
-<pinref part="SD" gate="A" pin="5"/>
+<pinref part="SPI" gate="A" pin="5"/>
 <wire x1="96.52" y1="-53.34" x2="104.14" y2="-53.34" width="0.1524" layer="91"/>
 <label x="88.9" y="-53.34" size="1.778" layer="95"/>
@@
 </segment>
 <segment>
-<pinref part="SD" gate="A" pin="6"/>
+<pinref part="SPI" gate="A" pin="6"/>
 <wire x1="96.52" y1="-55.88" x2="104.14" y2="-55.88" width="0.1524" layer="91"/>
 <label x="88.9" y="-55.88" size="1.778" layer="95"/>
@@
 </sheet>
 </sheets>
+<errors>
+</errors>
 </schematic>
 </drawing>
