File: clouds_v30.brd (EAGLE design)
At the start: 152.4 x 51.1 mm, 148 parts, among them IC1 74HC595D, IC10 TL072D, IC2 LM1117-3.3, IC3 MCP6002, IC4 MCP6004, IC5 STM32F405RGT6, IC6 LM4040B10, IC7 LM1117-3.3, IC8 WM8731, IC9 TL072D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

Commit message: almost all routed!
Parts:
- moved R57 1.00 mm to (1.59, 10.8)
- moved R46 0.95 mm to (1.59, 14.3)
- moved C12 0.45 mm to (80.0, 29.5)
- moved C14 0.45 mm to (81.0, 28.6)
Routing:
- net GND: track 213.5 -> 505.3 mm, vias 16 -> 24
- net PC6: track 60.5 -> 74.4 mm
- net N$58: track 4.04 -> 5.31 mm
- net N$21: track 8.74 -> 9.55 mm

Commit message: more routing! GRNDS!!!
Parts:
- moved C39 0.32 mm to (25.1, 16.5)
Routing:
- net GND: track 505.3 -> 539.4 mm, vias 24 -> 28
- net N$33: track 22.5 -> 14.8 mm, vias 0 -> 2
- net N$31: track 44.3 -> 47.1 mm
- net VCC: track 73.0 -> 74.1 mm

Commit message: everything is routed except a few grounds i think!
Routing:
- net GND: track 539.4 -> 661.4 mm, vias 28 -> 40
- net I2S_SOUT: track 0.00 -> 76.1 mm, vias 0 -> 4
- net RIN: track 17.1 -> 12.2 mm
- net +3V3_A: track 144.9 -> 147.9 mm
- net I2S_SIN: track 68.4 -> 65.5 mm
- net LIN: track 16.2 -> 18.2 mm
- net PC6: track 74.4 -> 72.8 mm
- net I2S_SCK: track 74.3 -> 75.2 mm
- net +3V3: track 342.8 -> 343.3 mm
- net I2S_LRCK: track 62.3 -> 61.7 mm

Commit message: completely routed!!! [i think, some weird unrouted stuff under pads]
Parts:
- moved C21 0.39 mm to (73.4, 23.9)
- moved R37 0.39 mm to (73.4, 20.7)
- moved R35 0.39 mm to (73.4, 22.3)
- moved R39 0.39 mm to (73.4, 19.1)
Routing:
- net GND: track 661.4 -> 734.8 mm, vias 40 -> 46
- net +3V3: track 343.3 -> 346.1 mm, vias 1 -> 3
- net AREF_-10: track 76.1 -> 76.7 mm

Commit message: added a bunch more documentation
Parts:
- moved C23 0.58 mm to (69.9, 22.9)
Routing:
- net GND: track 734.8 -> 736.8 mm
- net VEE: track 88.2 -> 86.5 mm
- net BLEND_CV: track 26.9 -> 25.8 mm
- net N$31: track 47.1 -> 47.7 mm
Other:
- board text added: "+3v3,G,SS,SCK,MISO,MOSI"
- board text added: "+3v3_a,Sz,Tx,P,B,Gnd"
- board text added: "12/15 XNOR Moved POTS/Jacks off board [headers] added SPI/SD port added port to remap: LED_EN, LED_SCK, V_OCT, BLEND_CV, TEXT_POT, BLEND_POT so that SPI port can be exposed use ORIG_MAP for original, NEW_MAP for SPI needs software change"
- board text added: "GND closer to edge"
- board text added: "GND, SIG, +V"
- board text added: "RED"
- board text added: "green"
- board text added: "led,btn"
- board text added: "mode, load"
- board text added: "rec, play"
